File: v1-v2/hardware/toniebox-v1v2.kicad_sch (KiCad schematic)
At the start: 146 parts, among them K2 Micro_SD_Card_Det_Hirose_DM3CS, K4 B3B-ZR-SM4-TF, K7 Barrel_Jack_MountingPin, K8 B3B-PH-SM4-TB, K9 B3B-PH-SM4-TB, T11 FDV301N, T2 MMBT3904, T3 MMBT3904, T360 FDV301N, T4 FDV301N, T5 FDV301N, T6 FDV301N, T7 FDV301N, U1 TLV320DAC3100, U2 CC3200R1M2RGCR, U3 IS25LQ032B-JNLE, U300 LM3485MM, U4 MMA8451QT, U6 AP2114H-3.3TRG1, U7 BQ24400, U8 AP2112K-3.3, U9 AP2120N-1.8

Commit message: Chg - KiCAD upgrade, More components
Parts:
- added D101: SS14, Diode_SMD:D_SMA, symbol Device:D_Schottky
- added D102: SS15, symbol Simulation_SPICE:D
- added Q101: NSS40200L, symbol Simulation_SPICE:PNP
- added R101: 6k7, symbol Device:R
- added R102: 10k, symbol Device:R
- added R103: 750R, symbol Device:R
- D6: footprint (none) -> Diode_SMD:D_SMA
Connections:
- net GND: now also K7.2, R55.2, TP55.1, U4.7 (SA0), D102.2 (A); no longer C58.2, K8.2, R53.1, R55.1, TP6.1, U7.2 (VSS)
- net NTC: now reaches K8.1, TP45.1, U7.5 (TS)
- net NTC: now also R101.1
- net at TP46.1, U7.6 (RC): now also R102.2
- net at D6.2 (A): now also D101.2 (A)
- net at U7.1 (SNS): now also R103.1
- net at U7.7 (VCC): now also R101.2, R102.1
- net at K7.1: now also D102.1 (K)
- new net: D101.1 (K), Q101.3 (E)
- new net BAT-: C58.2, K8.2, R103.2, R53.1, R55.1, TP6.1, U7.2 (VSS)
Other:
- note added: "WE501 - ?"
- moved on the sheet: D301, D6, K7, K8, R305, R351, R353, R37, R55, R61, R?3, T4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
